File: Rokavevo.kicad_sch (KiCad schematic)
At the start: 45 parts, among them J1 AudioJack2_Ground_Switch, Q1 BC847, Q2 BC847, Q3 BC847, Q4 BC847, Q5 BC847, SW1 SW_Nidec_CAS-120A1, U1 LM358, U2 LM358, Y1 3579kHz

Commit message: Add files via upload
Parts:
- removed J1: AudioJack2_Ground_Switch, Connector_Audio:Jack_3.5mm_CUI_SJ1-3515N_Horizontal, symbol Connector_Audio:AudioJack2_Ground_Switch
- added J2: AudioJack3_SwitchTR, Connector_Audio:Jack_3.5mm_CUI_SJ1-3515N_Horizontal, symbol Connector_Audio:AudioJack3_SwitchTR
Connections:
- net GND: now also J2.S
- net at C13.2: now also J2.R, J2.RN, J2.T, J2.TN
- net at C12.1: now also RV1.1; no longer RV1.3
- net at U1.1, U1.5 (+): now also RV1.3; no longer RV1.1
Other:
- moved on the sheet: RV1
Changed lines of the file:
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@@
 	)
 	(junction
-		(at 228.6 68.58)
-		(diameter 0)
-		(color 0 0 0 0)
-	)
-	(junction
 		(at 115.57 41.91)
 		(diameter 0)
@@
 	)
 	(junction
+		(at 228.6 63.5)
+		(diameter 0)
+		(color 0 0 0 0)
+	)
+	(junction
 		(at 198.12 60.96)
 		(diameter 0)
@@
 	)
 	(junction
+		(at 228.6 66.04)
+		(diameter 0)
+		(color 0 0 0 0)
+	)
+	(junction
 		(at 93.98 67.31)
 		(diameter 0)
@@
 	)
 	(junction
-		(at 58.42 41.91)
+		(at 228.6 68.58)
 		(diameter 0)
 		(color 0 0 0 0)
 	)
 	(junction
-		(at 132.08 52.07)
+		(at 58.42 41.91)
 		(diameter 0)
 		(color 0 0 0 0)
 	)
 	(junction
-		(at 228.6 63.5)
+		(at 132.08 52.07)
 		(diameter 0)
 		(color 0 0 0 0)
@@
 	)
 	(junction
-		(at 228.6 66.04)
-		(diameter 0)
-		(color 0 0 0 0)
-	)
-	(junction
 		(at 73.66 59.69)
 		(diameter 0)
@@
 	(wire
 		(pts
+			(xy 228.6 66.04) (xy 228.6 68.58)
+		)
+		(stroke
+			(width 0)
+			(type default)
+		)
+	)
+	(wire
+		(pts
 			(xy 157.48 109.22) (xy 111.76 109.22)
 		)
@@
 	(wire
 		(pts
+			(xy 227.33 60.96) (xy 228.6 60.96)
+		)
+		(stroke
+			(width 0)
+			(type default)
+		)
+	)
+	(wire
+		(pts
 			(xy 110.49 52.07) (xy 132.08 52.07)
 		)
@@
 	(wire
 		(pts
+			(xy 228.6 68.58) (xy 228.6 71.12)
+		)
+		(stroke
+			(width 0)
+			(type default)
+		)
+	)
+	(wire
+		(pts
 			(xy 111.76 109.22) (xy 111.76 67.31)
 		)
@@
 	(wire
 		(pts
-			(xy 228.6 68.58) (xy 228.6 71.12)
-		)
-		(stroke
-			(width 0)
-			(type default)
-		)
-	)
-	(wire
-		(pts
 			(xy 111.76 67.31) (xy 115.57 67.31)
 		)
@@
 	(wire
 		(pts
-			(xy 228.6 66.04) (xy 228.6 68.58)
-		)
-		(stroke
-			(width 0)
-			(type default)
-		)
-	)
-	(wire
-		(pts
 			(xy 147.32 68.58) (xy 149.86 68.58)
 		)
@@
 	(symbol
 		(lib_id "Device:R_Potentiometer")
-		(at 198.12 76.2 0)
-		(mirror y)
+		(at 198.12 76.2 180)
 		(unit 1)
 		(exclude_from_sim no)
@@
 		(dnp no)
 		(property "Reference" "RV1"
-			(at 201.168 75.946 0)
+			(at 201.168 76.454 0)
 			(effects
 				(font
@@
 		)
 		(property "Value" "R_Potentiometer"
-			(at 201.168 78.486 0)
+			(at 201.168 73.914 0)
 			(effects
 				(font
@@
 	(symbol
 		(lib_id "power:GND")
-		(at 233.68 76.2 0)
+		(at 227.33 60.96 270)
 		(unit 1)
 		(exclude_from_sim no)
@@
 		(fields_autoplaced yes)
 		(property "Reference" "#PWR013"
-			(at 233.68 82.55 0)
+			(at 220.98 60.96 0)
 			(effects
 				(font
@@
 		)
 		(property "Value" "GND"
-			(at 233.68 81.28 0)
+			(at 223.52 60.9599 90)
 			(effects
 				(font
 					(size 1.27 1.27)
 				)
+				(justify right)
 			)
 		)
 		(property "Footprint" ""
-			(at 233.68 76.2 0)
+			(at 227.33 60.96 0)
 			(effects
 				(font
@@
 		)
 		(property "Datasheet" ""
-			(at 233.68 76.2 0)
+			(at 227.33 60.96 0)
 			(effects
 				(font
@@
 		)
 		(property "Description" "Power symbol creates a global label with name \"GND\" , ground"
-			(at 233.68 76.2 0)
+			(at 227.33 60.96 0)
 			(effects
 				(font
@@
 	)
 	(symbol
-		(lib_id "Connector_Audio:AudioJack2_Ground_Switch")
-		(at 233.68 68.58 0)
-		(mirror y)
-		(unit 1)
-		(exclude_from_sim no)
-		(in_bom yes)
-		(on_board yes)
-		(dnp no)
-		(fields_autoplaced yes)
-		(property "Reference" "J1"
-			(at 238.76 66.6749 0)
-			(effects
-				(font
-					(size 1.27 1.27)
-				)
-				(justify right)
-			)
-		)
-		(property "Value" "AudioJack2_Ground_Switch"
-			(at 238.76 69.2149 0)
-			(effects
-				(font
-					(size 1.27 1.27)
-				)
-				(justify right)
-			)
-		)
-		(property "Footprint" "Connector_Audio:Jack_3.5mm_CUI_SJ1-3515N_Horizontal"
-			(at 233.68 63.5 0)
-			(effects
-				(font
-					(size 1.27 1.27)
-				)
-				(hide yes)
-			)
-		)
-		(property "Datasheet" "~"
-			(at 233.68 63.5 0)
-			(effects
-				(font
-					(size 1.27 1.27)
-				)
-				(hide yes)
-			)
-		)
-		(property "Description" "Audio Jack, 2 Poles (Mono / TS), Grounded Sleeve, Switched Pole (Normalling)"
-			(at 233.68 68.58 0)
-			(effects
-				(font
-					(size 1.27 1.27)
-				)
-				(hide yes)
-			)
-		)
-		(pin "S"
-		)
-		(pin "G"
-		)
-		(pin "SN"
-		)
-		(pin "T"
-		)
-		(pin "TN"
-		)
-		(instances
-			(project ""
-				(path "/bbb3eec1-57c2-4f73-8019-dc4bbdafbca9"
-					(reference "J1")
-					(unit 1)
-				)
-			)
-		)
-	)
-	(symbol
 		(lib_id "Device:R")
 		(at 119.38 67.31 90)
@@
 					(unit 1)
 				)
+			)
+		)
+	)
+	(symbol
+		(lib_id "Connector_Audio:AudioJack3_SwitchTR")
+		(at 233.68 63.5 0)
+		(mirror y)
+		(unit 1)
+		(exclude_from_sim no)
+		(in_bom yes)
+		(on_board yes)
+		(dnp no)
+		(property "Reference" "J2"
+			(at 235.585 54.61 0)
+			(effects
+				(font
+					(size 1.27 1.27)
+				)
+			)
+		)
+		(property "Value" "AudioJack3_SwitchTR"
+			(at 235.585 57.15 0)
+			(effects
+				(font
+					(size 1.27 1.27)
+				)
+			)
+		)
+		(property "Footprint" "Connector_Audio:Jack_3.5mm_CUI_SJ1-3515N_Horizontal"
+			(at 233.68 63.5 0)
+			(effects
+				(font
+					(size 1.27 1.27)
+				)
+				(hide yes)
+			)
+		)
+		(property "Datasheet" "~"
+			(at 233.68 63.5 0)
+			(effects
+				(font
+					(size 1.27 1.27)
+				)
+				(hide yes)
+			)
+		)
+		(property "Description" "Audio Jack, 3 Poles (Stereo / TRS), Switched TR Poles (Normalling)"
+			(at 233.68 63.5 0)
+			(effects
+				(font
+					(size 1.27 1.27)
+				)
+				(hide yes)
+			)
+		)
+		(pin "T"
+		)
+		(pin "S"
+		)
+		(pin "TN"
+		)
+		(pin "R"
+		)
+		(pin "RN"
+		)
+		(instances
+			(project ""
+				(path "/bbb3eec1-57c2-4f73-8019-dc4bbdafbca9"
+					(reference "J2")
+					(unit 1)
+				)

Commit message: Add files via upload
Parts:
- RV1: footprint Connector_PinHeader_2.54mm:PinHeader_1x03_P2.54mm_Vertical -> Potentiometer_THT:Potentiometer_Omeg_PC16BU_Vertical
Changed lines of the file:
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@@
 			)
 		)
-		(property "Footprint" "Connector_PinHeader_2.54mm:PinHeader_1x03_P2.54mm_Vertical"
+		(property "Footprint" "Potentiometer_THT:Potentiometer_Omeg_PC16BU_Vertical"
 			(at 198.12 76.2 0)
 			(effects

Commit message: Prototype II
Fixed schematic, new pcb design, Printable mask
Parts:
- C1, C12, C13: footprint Capacitor_SMD:C_0805_2012Metric_Pad1.18x1.45mm_HandSolder -> Capacitor_SMD:CP_Elec_6.3x5.3
- C3: footprint Capacitor_SMD:C_0805_2012Metric_Pad1.18x1.45mm_HandSolder -> Capacitor_SMD:C_1206_3216Metric_Pad1.33x1.80mm_HandSolder
- C5, C6, C7, C8: value 223 -> 181; footprint Capacitor_SMD:C_0805_2012Metric_Pad1.18x1.45mm_HandSolder -> Capacitor_SMD:C_1206_3216Metric_Pad1.33x1.80mm_HandSolder
Connections:
- net SBM: no longer C9.2, Q2.3 (C), R9.1
- net at Q1.3 (C), R3.2: now also C5.2; no longer C5.1
- net at C6.1, Q4.3 (C), R5.2: no longer C5.2, Q2.1 (B), R7.2
- new net: C5.1, Q2.1 (B), R7.2
- new net: C9.2, Q2.3 (C), R9.1
Other:
- moved on the sheet: C5, Q2
Changed lines of the file:
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@@
 	)
 	(junction
-		(at 102.87 57.15)
-		(diameter 0)
-		(color 0 0 0 0)
-	)
-	(junction
 		(at 102.87 52.07)
 		(diameter 0)
@@
 	)
 	(junction
-		(at 137.16 52.07)
-		(diameter 0)
-		(color 0 0 0 0)
-	)
-	(junction
 		(at 139.7 83.82)
 		(diameter 0)
@@
 	)
 	(junction
+		(at 132.08 53.34)
+		(diameter 0)
+		(color 0 0 0 0)
+	)
+	(junction
 		(at 115.57 74.93)
 		(diameter 0)
@@
 	)
 	(junction
+		(at 86.36 55.88)
+		(diameter 0)
+		(color 0 0 0 0)
+	)
+	(junction
 		(at 228.6 66.04)
 		(diameter 0)
@@
 	)
 	(junction
-		(at 132.08 52.07)
-		(diameter 0)
-		(color 0 0 0 0)
-	)
-	(junction
 		(at 157.48 58.42)
 		(diameter 0)
@@
 	)
 	(junction
-		(at 86.36 57.15)
+		(at 123.19 59.69)
 		(diameter 0)
 		(color 0 0 0 0)
@@
 	)
 	(junction
-		(at 123.19 57.15)
-		(diameter 0)
-		(color 0 0 0 0)
-	)
-	(junction
 		(at 115.57 67.31)
 		(diameter 0)
@@
 	(wire
 		(pts
-			(xy 93.98 57.15) (xy 102.87 57.15)
-		)
-		(stroke
-			(width 0)
-			(type default)
-		)
-	)
-	(wire
-		(pts
-			(xy 132.08 49.53) (xy 132.08 52.07)
-		)
-		(stroke
-			(width 0)
-			(type default)
-		)
-	)
-	(wire
-		(pts
-			(xy 137.16 52.07) (xy 157.48 52.07)
+			(xy 110.49 62.23) (xy 110.49 82.55)
 		)
 		(stroke
@@
 	(wire
 		(pts
-			(xy 110.49 62.23) (xy 110.49 82.55)
+			(xy 86.36 41.91) (xy 102.87 41.91)
 		)
 		(stroke
@@
 	(wire
 		(pts
-			(xy 86.36 41.91) (xy 102.87 41.91)
+			(xy 132.08 68.58) (xy 147.32 68.58)
 		)
 		(stroke
@@
 	(wire
 		(pts
-			(xy 132.08 68.58) (xy 147.32 68.58)
+			(xy 198.12 60.96) (xy 198.12 72.39)
 		)
 		(stroke
@@
 	(wire
 		(pts
-			(xy 198.12 60.96) (xy 198.12 72.39)
+			(xy 102.87 41.91) (xy 115.57 41.91)
 		)
 		(stroke
@@
 	(wire
 		(pts
-			(xy 102.87 41.91) (xy 115.57 41.91)
+			(xy 58.42 41.91) (xy 73.66 41.91)
 		)
 		(stroke
@@
 	(wire
 		(pts
-			(xy 58.42 41.91) (xy 73.66 41.91)
+			(xy 215.9 74.93) (xy 215.9 63.5)
 		)
 		(stroke
@@
 	(wire
 		(pts
-			(xy 215.9 74.93) (xy 215.9 63.5)
+			(xy 137.16 53.34) (xy 132.08 53.34)
 		)
 		(stroke
@@
 	(wire
 		(pts
-			(xy 123.19 57.15) (xy 124.46 57.15)
+			(xy 123.19 59.69) (xy 124.46 59.69)
 		)
 		(stroke
@@
 	(wire
 		(pts
-			(xy 137.16 52.07) (xy 137.16 55.88)
-		)
-		(stroke
-			(width 0)
-			(type default)
-		)
-	)
-	(wire
-		(pts
-			(xy 102.87 57.15) (xy 123.19 57.15)
-		)
-		(stroke
-			(width 0)
-			(type default)
-		)
-	)
-	(wire
-		(pts
 			(xy 129.54 74.93) (xy 133.35 74.93)
 		)
@@
 	(wire
 		(pts
-			(xy 110.49 52.07) (xy 132.08 52.07)
+			(xy 110.49 52.07) (xy 157.48 52.07)
 		)
 		(stroke
@@
 	(wire
 		(pts
-			(xy 132.08 52.07) (xy 137.16 52.07)
+			(xy 55.88 59.69) (xy 62.23 59.69)
 		)
 		(stroke
@@
 	(wire
 		(pts
-			(xy 55.88 59.69) (xy 62.23 59.69)
+			(xy 62.23 82.55) (xy 110.49 82.55)
 		)
 		(stroke
@@
 	(wire
 		(pts
-			(xy 62.23 82.55) (xy 110.49 82.55)
+			(xy 115.57 101.6) (xy 115.57 100.33)
 		)
 		(stroke
@@
 	(wire
 		(pts
-			(xy 115.57 101.6) (xy 115.57 100.33)
+			(xy 223.52 63.5) (xy 228.6 63.5)
 		)
 		(stroke
@@
 	(wire
 		(pts
-			(xy 223.52 63.5) (xy 228.6 63.5)
+			(xy 73.66 59.69) (xy 73.66 62.23)
 		)
 		(stroke
@@
 	(wire
 		(pts
-			(xy 73.66 59.69) (xy 73.66 62.23)
+			(xy 132.08 49.53) (xy 132.08 53.34)
 		)
 		(stroke
@@
 	(wire
 		(pts
-			(xy 73.66 62.23) (xy 73.66 64.77)
+			(xy 123.19 59.69) (xy 123.19 67.31)
 		)
 		(stroke
@@
 	(wire
 		(pts
-			(xy 186.69 41.91) (xy 204.47 41.91)
+			(xy 73.66 62.23) (xy 73.66 64.77)
 		)
 		(stroke
@@
 	(wire
 		(pts
-			(xy 132.08 52.07) (xy 132.08 53.34)
+			(xy 186.69 41.91) (xy 204.47 41.91)
 		)
 		(stroke
@@
 	(wire
 		(pts
+			(xy 93.98 55.88) (xy 123.19 55.88)
+		)
+		(stroke
+			(width 0)
+			(type default)
+		)
+	)
+	(wire
+		(pts
 			(xy 172.72 58.42) (xy 172.72 62.23)
 		)
@@
 	(wire
 		(pts
-			(xy 86.36 49.53) (xy 86.36 57.15)
+			(xy 86.36 49.53) (xy 86.36 55.88)
 		)
 		(stroke
@@
 	(wire
 		(pts
-			(xy 123.19 57.15) (xy 123.19 67.31)
+			(xy 123.19 55.88) (xy 123.19 59.69)
 		)
 		(stroke
@@
 	(wire
 		(pts
+			(xy 132.08 53.34) (xy 132.08 54.61)
+		)
+		(stroke
+			(width 0)
+			(type default)
+		)
+	)
+	(wire
+		(pts
 			(xy 147.32 80.01) (xy 147.32 83.82)
 		)
@@
 	(wire
 		(pts
-			(xy 132.08 62.23) (xy 132.08 68.58)
+			(xy 132.08 64.77) (xy 132.08 68.58)
+		)
+		(stroke
+			(width 0)
+			(type default)
+		)
+	)
+	(wire
+		(pts
+			(xy 86.36 55.88) (xy 86.36 57.15)
+		)
+		(stroke
+			(width 0)
+			(type default)
+		)
+	)
+	(wire
+		(pts
+			(xy 137.16 55.88) (xy 137.16 53.34)
 		)
 		(stroke
@@
 			)
 		)
-		(property "Footprint" "Capacitor_SMD:C_0805_2012Metric_Pad1.18x1.45mm_HandSolder"
+		(property "Footprint" "Capacitor_SMD:CP_Elec_6.3x5.3"
 			(at 223.52 62.5348 0)
 			(effects
@@
 	(symbol
 		(lib_id "Device:C")
-		(at 90.17 57.15 90)
+		(at 90.17 55.88 270)
+		(mirror x)
 		(unit 1)
 		(exclude_from_sim no)
@@
 		(dnp no)
 		(property "Reference" "C5"
-			(at 93.98 54.864 90)
+			(at 86.36 53.594 90)
 			(effects
 				(font
@@
 			)
 		)
-		(property "Value" "223"
-			(at 90.17 52.832 90)
+		(property "Value" "181"
+			(at 90.17 51.562 90)
 			(effects
 				(font
@@
 			)
 		)
-		(property "Footprint" "Capacitor_SMD:C_0805_2012Metric_Pad1.18x1.45mm_HandSolder"
-			(at 93.98 56.1848 0)
+		(property "Footprint" "Capacitor_SMD:C_1206_3216Metric_Pad1.33x1.80mm_HandSolder"
+			(at 86.36 54.9148 0)
 			(effects
 				(font
@@
 		)
 		(property "Datasheet" "~"
-			(at 90.17 57.15 0)
+			(at 90.17 55.88 0)
 			(effects
 				(font
@@
 		)
 		(property "Description" "Unpolarized capacitor"
-			(at 90.17 57.15 0)
+			(at 90.17 55.88 0)
 			(effects
 				(font
@@
 	(symbol
 		(lib_id "Transistor_BJT:BC847")
-		(at 129.54 57.15 0)
+		(at 129.54 59.69 0)
 		(unit 1)
 		(exclude_from_sim no)
@@
 		(dnp no)
 		(property "Reference" "Q2"
-			(at 127 53.594 0)
+			(at 127 56.134 0)
 			(effects
 				(font
@@
 		)
 		(property "Value" "BC847"
-			(at 125.222 62.484 0)
+			(at 125.222 65.024 0)
 			(effects
 				(font
@@
 		)
 		(property "Footprint" "Package_TO_SOT_SMD:SOT-23"
-			(at 134.62 59.055 0)
+			(at 134.62 61.595 0)
 			(effects
 				(font
@@
 		)
 		(property "Datasheet" "http://www.infineon.com/dgdl/Infineon-BC847SERIES_BC848SERIES_BC849SERIES_BC850SERIES-DS-v01_01-en.pdf?fileId=db3a304314dca389011541d4630a1657"
-			(at 129.54 57.15 0)
+			(at 129.54 59.69 0)
 			(effects
 				(font
@@
 		)
 		(property "Description" "0.1A Ic, 45V Vce, NPN Transistor, SOT-23"
-			(at 129.54 57.15 0)
+			(at 129.54 59.69 0)
 			(effects
 				(font
@@
 			)
 		)
-		(property "Footprint" "Capacitor_SMD:C_0805_2012Metric_Pad1.18x1.45mm_HandSolder"
+		(property "Footprint" "Capacitor_SMD:CP_Elec_6.3x5.3"
 			(at 199.0852 87.63 0)
 			(effects
@@
 			)
 		)
-		(property "Value" "223"
+		(property "Value" "181"
 			(at 139.7 93.218 0)
 			(effects
@@
 			)
 		)
-		(property "Footprint" "Capacitor_SMD:C_0805_2012Metric_Pad1.18x1.45mm_HandSolder"
+		(property "Footprint" "Capacitor_SMD:C_1206_3216Metric_Pad1.33x1.80mm_HandSolder"
 			(at 138.7348 86.36 0)
 			(effects
@@
 			)
 		)
-		(property "Value" "223"
+		(property "Value" "181"
 			(at 141.732 80.264 0)
 			(effects
@@
 			)
 		)
-		(property "Footprint" "Capacitor_SMD:C_0805_2012Metric_Pad1.18x1.45mm_HandSolder"
+		(property "Footprint" "Capacitor_SMD:C_1206_3216Metric_Pad1.33x1.80mm_HandSolder"
 			(at 138.7348 74.93 0)
 			(effects
@@
 			)
 		)
-		(property "Value" "223"
+		(property "Value" "181"
 			(at 109.22 50.546 90)
 			(effects
@@
 			)
 		)
-		(property "Footprint" "Capacitor_SMD:C_0805_2012Metric_Pad1.18x1.45mm_HandSolder"
+		(property "Footprint" "Capacitor_SMD:C_1206_3216Metric_Pad1.33x1.80mm_HandSolder"
 			(at 110.49 51.1048 0)
 			(effects
@@
 			)
 		)
-		(property "Footprint" "Capacitor_SMD:C_0805_2012Metric_Pad1.18x1.45mm_HandSolder"
+		(property "Footprint" "Capacitor_SMD:C_1206_3216Metric_Pad1.33x1.80mm_HandSolder"
 			(at 63.1952 67.31 0)
 			(effects
@@
 			)
 		)
-		(property "Footprint" "Capacitor_SMD:C_0805_2012Metric_Pad1.18x1.45mm_HandSolder"
+		(property "Footprint" "Capacitor_SMD:CP_Elec_6.3x5.3"
 			(at 49.2252 49.53 0)
 			(effects
